File: SpectrumAnalyzer.sch (KiCad schematic (older format))
At the start: 183 parts, among them J1 Conn_01x03_Male, J2 Conn_01x03_Male

Commit message: minor updates
Parts:
- D1: LCSC (none) -> C114586
Changed lines of the file:
@@
 F 2 "LED_SMD:LED_WS2812B_PLCC4_5.0x5.0mm_P3.2mm" H 1950 1300 50  0001 L TNN
 F 3 "https://cdn-shop.adafruit.com/datasheets/WS2812B.pdf" H 2000 1225 50  0001 L TNN
+F 4 "C114586" H 1900 1600 50  0001 C CNN "LCSC"
 	1    1900 1600
 	1    0    0    -1
